File: cad/sumo2/sumo2.kicad_sch (KiCad schematic)
At the start: 15 parts, among them M1 Motor_DC, M2 Motor_DC, M3 Motor_DC, M4 Motor_DC, P1 Raspi 4B Pin Headers, U1 SF Motor Driver Board, U2 SF Motor Driver Board

Commit message: schematic rev 2.1
Parts:
- removed A1: Redboard, Module:Arduino_UNO_R3, symbol MCU_Module:Arduino_UNO_R3
- added V1: 5V Regulator, symbol sf:Voltage_Regulator
Connections:
- net +3V3: now also P1.1 (Pin_1)
- net +5V: now also V1. (VIN-)
- net Earth: now also V1. (VIN-); no longer BT2.2 (-)
- net +BATT renamed +6V
- net A1_JACK: no longer names the net of BT2.1 (+)
- net A1_JACK: now also V1. (VIN-)
- new net: BT2.2 (-), V1. (VIN-)
- no-connect marks 47 -> 18
Other:
- note added: "4 Alkaline AA (6V)"
- note added: "8 Alkaline AA (12V)"
- note removed: "4 Alkaline AA"
- note removed: "6 NiCd Rechargable AA"
- moved on the sheet: BT1, BT2
